File: Hardware/MoodBadge.sch (EAGLE design)
At the start: 1 part

Commit message: EAGLE files
Parts:
- removed D1: 15KEXX, diode:15KEXX
Changed lines of the file:
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@@
 <grid distance="0.1" unitdist="inch" unit="inch" style="lines" multiple="1" display="no" altdistance="0.01" altunitdist="inch" altunit="inch"/>
 <layers>
-<layer number="1" name="Top" color="4" fill="1" visible="no" active="no"/>
-<layer number="2" name="Route2" color="1" fill="3" visible="no" active="no"/>
-<layer number="3" name="Route3" color="4" fill="3" visible="no" active="no"/>
-<layer number="4" name="Route4" color="1" fill="4" visible="no" active="no"/>
-<layer number="5" name="Route5" color="4" fill="4" visible="no" active="no"/>
-<layer number="6" name="Route6" color="1" fill="8" visible="no" active="no"/>
-<layer number="7" name="Route7" color="4" fill="8" visible="no" active="no"/>
-<layer number="8" name="Route8" color="1" fill="2" visible="no" active="no"/>
-<layer number="9" name="Route9" color="4" fill="2" visible="no" active="no"/>
-<layer number="10" name="Route10" color="1" fill="7" visible="no" active="no"/>
-<layer number="11" name="Route11" color="4" fill="7" visible="no" active="no"/>
-<layer number="12" name="Route12" color="1" fill="5" visible="no" active="no"/>
-<layer number="13" name="Route13" color="4" fill="5" visible="no" active="no"/>
-<layer number="14" name="Route14" color="1" fill="6" visible="no" active="no"/>
-<layer number="15" name="Route15" color="4" fill="6" visible="no" active="no"/>
-<layer number="16" name="Bottom" color="1" fill="1" visible="no" active="no"/>
-<layer number="17" name="Pads" color="2" fill="1" visible="no" active="no"/>
-<layer number="18" name="Vias" color="2" fill="1" visible="no" active="no"/>
-<layer number="19" name="Unrouted" color="6" fill="1" visible="no" active="no"/>
-<layer number="20" name="Dimension" color="15" fill="1" visible="no" active="no"/>
-<layer number="21" name="tPlace" color="7" fill="1" visible="no" active="no"/>
-<layer number="22" name="bPlace" color="7" fill="1" visible="no" active="no"/>
-<layer number="23" name="tOrigins" color="15" fill="1" visible="no" active="no"/>
-<layer number="24" name="bOrigins" color="15" fill="1" visible="no" active="no"/>
-<layer number="25" name="tNames" color="7" fill="1" visible="no" active="no"/>
-<layer number="26" name="bNames" color="7" fill="1" visible="no" active="no"/>
-<layer number="27" name="tValues" color="7" fill="1" visible="no" active="no"/>
-<layer number="28" name="bValues" color="7" fill="1" visible="no" active="no"/>
-<layer number="29" name="tStop" color="7" fill="3" visible="no" active="no"/>
-<layer number="30" name="bStop" color="7" fill="6" visible="no" active="no"/>
-<layer number="31" name="tCream" color="7" fill="4" visible="no" active="no"/>
-<layer number="32" name="bCream" color="7" fill="5" visible="no" active="no"/>
-<layer number="33" name="tFinish" color="6" fill="3" visible="no" active="no"/>
-<layer number="34" name="bFinish" color="6" fill="6" visible="no" active="no"/>
-<layer number="35" name="tGlue" color="7" fill="4" visible="no" active="no"/>
-<layer number="36" name="bGlue" color="7" fill="5" visible="no" active="no"/>
-<layer number="37" name="tTest" color="7" fill="1" visible="no" active="no"/>
-<layer number="38" name="bTest" color="7" fill="1" visible="no" active="no"/>
-<layer number="39" name="tKeepout" color="4" fill="11" visible="no" active="no"/>
-<layer number="40" name="bKeepout" color="1" fill="11" visible="no" active="no"/>
-<layer number="41" name="tRestrict" color="4" fill="10" visible="no" active="no"/>
-<layer number="42" name="bRestrict" color="1" fill="10" visible="no" active="no"/>
-<layer number="43" name="vRestrict" color="2" fill="10" visible="no" active="no"/>
-<layer number="44" name="Drills" color="7" fill="1" visible="no" active="no"/>
-<layer number="45" name="Holes" color="7" fill="1" visible="no" active="no"/>
-<layer number="46" name="Milling" color="3" fill="1" visible="no" active="no"/>
-<layer number="47" name="Measures" color="7" fill="1" visible="no" active="no"/>
-<layer number="48" name="Document" color="7" fill="1" visible="no" active="no"/>
-<layer number="49" name="Reference" color="7" fill="1" visible="no" active="no"/>
-<layer number="51" name="tDocu" color="6" fill="1" visible="no" active="no"/>
-<layer number="52" name="bDocu" color="7" fill="1" visible="no" active="no"/>
 <layer number="88" name="SimResults" color="9" fill="1" visible="yes" active="yes"/>
 <layer number="89" name="SimProbes" color="9" fill="1" visible="yes" active="yes"/>
@@
 <layer number="97" name="Info" color="7" fill="1" visible="yes" active="yes"/>
 <layer number="98" name="Guide" color="6" fill="1" visible="yes" active="yes"/>
-<layer number="99" name="SpiceOrder" color="5" fill="1" visible="yes" active="yes"/>
 </layers>
 <schematic xreflabel="%F%N/%S.%C%R" xrefpart="/%S.%C%R">
@@
 </classes>
 <parts>
-<part name="D1" library="diode" library_urn="urn:adsk.eagle:library:210" deviceset="15KEXX" device="" package3d_urn="urn:adsk.eagle:package:43360/1"/>
 </parts>
 <sheets>
@@
 </plain>
 <instances>
-<instance part="D1" gate="1" x="50.8" y="60.96" smashed="yes">
-<attribute name="NAME" x="48.514" y="62.865" size="1.778" layer="95"/>
-<attribute name="VALUE" x="48.514" y="57.531" size="1.778" layer="96"/>
-</instance>
 </instances>
 <busses>
@@
 </schematic>
 </drawing>
-<compatibility>
-<note version="8.2" severity="warning">
-Since Version 8.2, EAGLE supports online libraries. The ids
-of those online libraries will not be understood (or retained)
-with this version.
-</note>
-<note version="8.3" severity="warning">
-Since Version 8.3, EAGLE supports URNs for individual library
-assets (packages, symbols, and devices). The URNs of those assets
-will not be understood (or retained) with this version.
-</note>
-<note version="8.3" severity="warning">
-Since Version 8.3, EAGLE supports the association of 3D packages
-with devices in libraries, schematics, and board files. Those 3D
-packages will not be understood (or retained) with this version.
-</note>
-</compatibility>
 </eagle>

Commit message: Created board outline and started schematic
Parts:
- added C1, C8, C9: 4.7uF, SparkFun-Capacitors:4.7UF-0603-6.3V-(10%)
- added C2, C3, C4, C5, C6, C7: 100n, LinnesLab-Passives:CAPACITOR0603
- added D1, D2: 1A/23V/620mV, LinnesLab-DiscreteSemi:SCHOTTKY-USC
- added DOWN, LEFT, MODE, RIGHT, SELECT, UP: (no value), LinnesLab-Switches:SPST.KT11P4SM34LFS
- added LED1, LED2, LED3, LED4, LED5, LED6, LED7: (no value), LinnesLab-LED:LED0603
- added LIPO: (no value), LinnesLab-Connectors:JST_2MM_MALE
- added ON/OFF: SWITCH.JS202011JXQNUPWARDS, LinnesLab-Switches:SWITCH.JS202011JXQNUPWARDS
- added R1, R11, R3, R5, R7, R9: 10k, LinnesLab-Passives:RESISTOR0603
- added R10, R12, R13, R14, R2, R4, R6, R8: 1k, LinnesLab-Passives:RESISTOR0603
- added U1: MCP73831, SparkFun-IC-Power:MCP73831
Connections:
- new net DOWN: C4.1, DOWN.B, R5.2, R6.2
- new net GND: C1.2, C2.2, C3.2, C4.2, C5.2, C6.2, C7.2, C9.2, LED1.C, LED2.C, LED3.C, LED4.C, LED5.C, LED6.C, LIPO.-, R1.1, R11.1, R14.1, R3.1, R5.1, R7.1, R9.1, U1.VSS
- new net LEFT: C2.1, LEFT.B, R1.2, R2.2
- new net MODE: C7.1, MODE.B, R11.2, R12.2
- new net N$11: LED5.A, R10.1
- new net N$13: LED6.A, R12.1
- new net N$2: D1.A, ON/OFF.1
- new net N$3: LED1.A, R2.1
- new net N$4: R14.2, U1.PROG
- new net N$5: LED2.A, R4.1
- new net N$7: LED3.A, R6.1
- new net N$9: LED4.A, R8.1
- new net RIGHT: C6.1, R10.2, R9.2, RIGHT.B
- new net SELECT: C3.1, R3.2, R4.2, SELECT.B
- new net UP: C5.1, R7.2, R8.2, UP.B
- new net VCC: DOWN.A, LEFT.A, MODE.A, RIGHT.A, SELECT.A, UP.A
- new net VLIPO: C1.1, C9.1, D1.C, LIPO.+, ON/OFF.2, U1.VBAT
Other:
- note added: "Action Buttons"
- note added: "Battery Charger"
- note added: "Power and On/Off Switch"
