File: Hardware/MoodBadge.sch (EAGLE design)
At the start: 80 parts, among them IC1 PCF8574T, U2 ATMEGA328P_TQFP, Y1 Crystal-CA-310

Commit message: Changed heart rate LED to IR LED and moved closer to the photoresistor
Parts:
- LED8: device LinnesLab-LED:LED0603 -> LinnesLab-LED:LEDZ-BEND
Changed lines of the file:
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@@
 <part name="GND33" library="LinnesLab-Symbols" deviceset="GND" device=""/>
 <part name="SUPPLY17" library="LinnesLab-Symbols" deviceset="VCC" device=""/>
-<part name="LED8" library="LinnesLab-LED" deviceset="LED" device="0603" package3d_urn="urn:adsk.eagle:package:18593052/2"/>
+<part name="LED8" library="LinnesLab-LED" deviceset="LED" device="Z-BEND"/>
 <part name="R24" library="LinnesLab-Passives" deviceset="RESISTOR" device="0603" package3d_urn="urn:adsk.eagle:package:15661944/2" value="487"/>
 <part name="GND34" library="LinnesLab-Symbols" deviceset="GND" device=""/>
